Commit message: fix import and relative path

File: models/cad_models/urdf/blue_bin.urdf (robot description, URDF)
Before this commit: robot blue_bin, 1 links, 0 joints
Links:
- link blue_bin: geometry collision box size=0.27 0.36 0.02; collision box size=0.27 0.36 0.02

File: models/cad_models/urdf/door_h20.urdf (robot description, URDF)
Before this commit: robot door_h20, 3 links, 2 joints
Links:
- link base_link: geometry visual mesh filename=package://uwds3/models/cad_models/obj/door_h20.obj scale=1 1 1
- link door_h20_1: geometry visual mesh filename=package://uwds3/models/cad_models/obj/door_h20_1.obj scale=1 1 1
- link door_h20_2: geometry visual mesh filename=package://uwds3/models/cad_models/obj/door_h20_2.obj scale=1 1 1

File: models/cad_models/urdf/elevator_1.urdf (robot description, URDF)
Before this commit: robot elevator_1, 2 links, 1 joints
Links:
- link elevator: geometry visual mesh filename=package://uwds3/models/cad_models/obj/elevator_1.obj scale=1 0.9 1

File: models/cad_models/urdf/glass_door.urdf (robot description, URDF)
Before this commit: robot glass_door, 3 links, 2 joints
Links:
- link glass_door_1: geometry visual mesh filename=package://uwds3/models/cad_models/obj/glass_door_1.obj scale=1 1 1
- link glass_door_2: geometry visual mesh filename=package://uwds3/models/cad_models/obj/glass_door_2.obj scale=1 1 1

File: models/cad_models/urdf/green_bin.urdf (robot description, URDF)
Before this commit: robot green_bin, 1 links, 0 joints
Links:
- link green_bin: geometry collision box size=0.27 0.36 0.02; collision box size=0.27 0.36 0.02

File: models/cad_models/urdf/simple_door.urdf (robot description, URDF)
Before this commit: robot simple_door, 2 links, 1 joints
Links:
- link simple_door: geometry visual mesh filename=package://uwds3/models/cad_models/obj/simple_door.obj scale=1 1 1

File: models/cad_models/urdf/stairs_1.urdf (robot description, URDF)
Before this commit: robot stairs_1, 1 links, 0 joints
Links:
- link base_link: geometry visual mesh filename=package://uwds3/models/cad_models/obj/stairs_1.obj scale=1 1 1
