Commit message: prepare data generator and various fix

File: models/cad_models/urdf/adream_empty.urdf (robot description, URDF)
Before this commit: robot adream_empty, 7 links, 6 joints
Links:
- link base_link: geometry collision mesh filename=package://uwds3/models/cad_models/obj/walls.obj scale=1 1 1; visual mesh filename=package://uwds3/models/cad_models/obj/walls.obj scale=1 1 1
