Commit message: refactoring and diverse fixes

File: models/cad_models/urdf/pepper.urdf (robot description, URDF)
Before this commit: robot PepperLaasMove3d, 53 links, 52 joints
Links:
- link Head: geometry collision mesh filename=package://pepper_meshes/meshes/1.0/HeadPitch_0.10.stl scale=0.1 0.1 0.1; visual mesh filename=package://pepper_meshes/meshes/1.0/HeadPitch_0.10.stl scale=0.1 0.1 0.1
- link Hip: geometry collision mesh filename=package://pepper_meshes/meshes/1.0/HipRoll_0.10.stl scale=0.1 0.1 0.1; visual mesh filename=package://pepper_meshes/meshes/1.0/HipRoll_0.10.stl scale=0.1 0.1 0.1
- link LBicep: geometry collision mesh filename=package://pepper_meshes/meshes/1.0/LShoulderRoll_0.10.stl scale=0.1 0.1 0.1; visual mesh filename=package://pepper_meshes/meshes/1.0/LShoulderRoll_0.10.stl scale=0.1 0.1 0.1
- link LElbow: geometry collision mesh filename=package://pepper_meshes/meshes/1.0/LElbowYaw_0.10.stl scale=0.1 0.1 0.1; visual mesh filename=package://pepper_meshes/meshes/1.0/LElbowYaw_0.10.stl scale=0.1 0.1 0.1
- link LFinger11_link: geometry collision mesh filename=package://pepper_meshes/meshes/1.0/LFinger11_0.10.stl scale=0.1 0.1 0.1; visual mesh filename=package://pepper_meshes/meshes/1.0/LFinger11_0.10.stl scale=0.1 0.1 0.1
- link LFinger12_link: geometry collision mesh filename=package://pepper_meshes/meshes/1.0/LFinger12_0.10.stl scale=0.1 0.1 0.1; visual mesh filename=package://pepper_meshes/meshes/1.0/LFinger12_0.10.stl scale=0.1 0.1 0.1
- link LFinger13_link: geometry collision mesh filename=package://pepper_meshes/meshes/1.0/LFinger13_0.10.stl scale=0.1 0.1 0.1; visual mesh filename=package://pepper_meshes/meshes/1.0/LFinger13_0.10.stl scale=0.1 0.1 0.1
- link LFinger21_link: geometry collision mesh filename=package://pepper_meshes/meshes/1.0/LFinger21_0.10.stl scale=0.1 0.1 0.1; visual mesh filename=package://pepper_meshes/meshes/1.0/LFinger21_0.10.stl scale=0.1 0.1 0.1
- link LFinger22_link: geometry collision mesh filename=package://pepper_meshes/meshes/1.0/LFinger22_0.10.stl scale=0.1 0.1 0.1; visual mesh filename=package://pepper_meshes/meshes/1.0/LFinger22_0.10.stl scale=0.1 0.1 0.1
- link LFinger23_link: geometry collision mesh filename=package://pepper_meshes/meshes/1.0/LFinger23_0.10.stl scale=0.1 0.1 0.1; visual mesh filename=package://pepper_meshes/meshes/1.0/LFinger23_0.10.stl scale=0.1 0.1 0.1
- link LFinger31_link: geometry collision mesh filename=package://pepper_meshes/meshes/1.0/LFinger31_0.10.stl scale=0.1 0.1 0.1; visual mesh filename=package://pepper_meshes/meshes/1.0/LFinger31_0.10.stl scale=0.1 0.1 0.1
- link LFinger32_link: geometry collision mesh filename=package://pepper_meshes/meshes/1.0/LFinger32_0.10.stl scale=0.1 0.1 0.1; visual mesh filename=package://pepper_meshes/meshes/1.0/LFinger32_0.10.stl scale=0.1 0.1 0.1
- link LFinger33_link: geometry collision mesh filename=package://pepper_meshes/meshes/1.0/LFinger33_0.10.stl scale=0.1 0.1 0.1; visual mesh filename=package://pepper_meshes/meshes/1.0/LFinger33_0.10.stl scale=0.1 0.1 0.1
- link LFinger41_link: geometry collision mesh filename=package://pepper_meshes/meshes/1.0/LFinger41_0.10.stl scale=0.1 0.1 0.1; visual mesh filename=package://pepper_meshes/meshes/1.0/LFinger41_0.10.stl scale=0.1 0.1 0.1
- link LFinger42_link: geometry collision mesh filename=package://pepper_meshes/meshes/1.0/LFinger42_0.10.stl scale=0.1 0.1 0.1; visual mesh filename=package://pepper_meshes/meshes/1.0/LFinger42_0.10.stl scale=0.1 0.1 0.1
- link LFinger43_link: geometry collision mesh filename=package://pepper_meshes/meshes/1.0/LFinger43_0.10.stl scale=0.1 0.1 0.1; visual mesh filename=package://pepper_meshes/meshes/1.0/LFinger43_0.10.stl scale=0.1 0.1 0.1
- link LForeArm: geometry collision mesh filename=package://pepper_meshes/meshes/1.0/LElbowRoll_0.10.stl scale=0.1 0.1 0.1; visual mesh filename=package://pepper_meshes/meshes/1.0/LElbowRoll_0.10.stl scale=0.1 0.1 0.1
- link LShoulder: geometry collision mesh filename=package://pepper_meshes/meshes/1.0/LShoulderPitch_0.10.stl scale=0.1 0.1 0.1; visual mesh filename=package://pepper_meshes/meshes/1.0/LShoulderPitch_0.10.stl scale=0.1 0.1 0.1
- link LThumb1_link: geometry collision mesh filename=package://pepper_meshes/meshes/1.0/LThumb1_0.10.stl scale=0.1 0.1 0.1; visual mesh filename=package://pepper_meshes/meshes/1.0/LThumb1_0.10.stl scale=0.1 0.1 0.1
- link LThumb2_link: geometry collision mesh filename=package://pepper_meshes/meshes/1.0/LThumb2_0.10.stl scale=0.1 0.1 0.1; visual mesh filename=package://pepper_meshes/meshes/1.0/LThumb2_0.10.stl scale=0.1 0.1 0.1
- link Neck: geometry collision mesh filename=package://pepper_meshes/meshes/1.0/HeadYaw_0.10.stl scale=0.1 0.1 0.1; visual mesh filename=package://pepper_meshes/meshes/1.0/HeadYaw_0.10.stl scale=0.1 0.1 0.1
- link Pelvis: geometry collision mesh filename=package://pepper_meshes/meshes/1.0/HipPitch_0.10.stl scale=0.1 0.1 0.1; visual mesh filename=package://pepper_meshes/meshes/1.0/HipPitch_0.10.stl scale=0.1 0.1 0.1
- link RBicep: geometry collision mesh filename=package://pepper_meshes/meshes/1.0/RShoulderRoll_0.10.stl scale=0.1 0.1 0.1; visual mesh filename=package://pepper_meshes/meshes/1.0/RShoulderRoll_0.10.stl scale=0.1 0.1 0.1
- link RElbow: geometry collision mesh filename=package://pepper_meshes/meshes/1.0/RElbowYaw_0.10.stl scale=0.1 0.1 0.1; visual mesh filename=package://pepper_meshes/meshes/1.0/RElbowYaw_0.10.stl scale=0.1 0.1 0.1
- link RFinger11_link: geometry collision mesh filename=package://pepper_meshes/meshes/1.0/RFinger11_0.10.stl scale=0.1 0.1 0.1; visual mesh filename=package://pepper_meshes/meshes/1.0/RFinger11_0.10.stl scale=0.1 0.1 0.1
- link RFinger12_link: geometry collision mesh filename=package://pepper_meshes/meshes/1.0/RFinger12_0.10.stl scale=0.1 0.1 0.1; visual mesh filename=package://pepper_meshes/meshes/1.0/RFinger12_0.10.stl scale=0.1 0.1 0.1
- link RFinger13_link: geometry collision mesh filename=package://pepper_meshes/meshes/1.0/RFinger13_0.10.stl scale=0.1 0.1 0.1; visual mesh filename=package://pepper_meshes/meshes/1.0/RFinger13_0.10.stl scale=0.1 0.1 0.1
- link RFinger21_link: geometry collision mesh filename=package://pepper_meshes/meshes/1.0/RFinger21_0.10.stl scale=0.1 0.1 0.1; visual mesh filename=package://pepper_meshes/meshes/1.0/RFinger21_0.10.stl scale=0.1 0.1 0.1
- link RFinger22_link: geometry collision mesh filename=package://pepper_meshes/meshes/1.0/RFinger22_0.10.stl scale=0.1 0.1 0.1; visual mesh filename=package://pepper_meshes/meshes/1.0/RFinger22_0.10.stl scale=0.1 0.1 0.1
- link RFinger23_link: geometry collision mesh filename=package://pepper_meshes/meshes/1.0/RFinger23_0.10.stl scale=0.1 0.1 0.1; visual mesh filename=package://pepper_meshes/meshes/1.0/RFinger23_0.10.stl scale=0.1 0.1 0.1
- link RFinger31_link: geometry collision mesh filename=package://pepper_meshes/meshes/1.0/RFinger31_0.10.stl scale=0.1 0.1 0.1; visual mesh filename=package://pepper_meshes/meshes/1.0/RFinger31_0.10.stl scale=0.1 0.1 0.1
- link RFinger32_link: geometry collision mesh filename=package://pepper_meshes/meshes/1.0/RFinger32_0.10.stl scale=0.1 0.1 0.1; visual mesh filename=package://pepper_meshes/meshes/1.0/RFinger32_0.10.stl scale=0.1 0.1 0.1
- link RFinger33_link: geometry collision mesh filename=package://pepper_meshes/meshes/1.0/RFinger33_0.10.stl scale=0.1 0.1 0.1; visual mesh filename=package://pepper_meshes/meshes/1.0/RFinger33_0.10.stl scale=0.1 0.1 0.1
- link RFinger41_link: geometry collision mesh filename=package://pepper_meshes/meshes/1.0/RFinger41_0.10.stl scale=0.1 0.1 0.1; visual mesh filename=package://pepper_meshes/meshes/1.0/RFinger41_0.10.stl scale=0.1 0.1 0.1
- link RFinger42_link: geometry collision mesh filename=package://pepper_meshes/meshes/1.0/RFinger42_0.10.stl scale=0.1 0.1 0.1; visual mesh filename=package://pepper_meshes/meshes/1.0/RFinger42_0.10.stl scale=0.1 0.1 0.1
- link RFinger43_link: geometry collision mesh filename=package://pepper_meshes/meshes/1.0/RFinger43_0.10.stl scale=0.1 0.1 0.1; visual mesh filename=package://pepper_meshes/meshes/1.0/RFinger43_0.10.stl scale=0.1 0.1 0.1
- link RForeArm: geometry collision mesh filename=package://pepper_meshes/meshes/1.0/RElbowRoll_0.10.stl scale=0.1 0.1 0.1; visual mesh filename=package://pepper_meshes/meshes/1.0/RElbowRoll_0.10.stl scale=0.1 0.1 0.1
- link RShoulder: geometry collision mesh filename=package://pepper_meshes/meshes/1.0/RShoulderPitch_0.10.stl scale=0.1 0.1 0.1; visual mesh filename=package://pepper_meshes/meshes/1.0/RShoulderPitch_0.10.stl scale=0.1 0.1 0.1
- link RThumb1_link: geometry collision mesh filename=package://pepper_meshes/meshes/1.0/RThumb1_0.10.stl scale=0.1 0.1 0.1; visual mesh filename=package://pepper_meshes/meshes/1.0/RThumb1_0.10.stl scale=0.1 0.1 0.1
- link RThumb2_link: geometry collision mesh filename=package://pepper_meshes/meshes/1.0/RThumb2_0.10.stl scale=0.1 0.1 0.1; visual mesh filename=package://pepper_meshes/meshes/1.0/RThumb2_0.10.stl scale=0.1 0.1 0.1
- link Tibia: geometry collision mesh filename=package://pepper_meshes/meshes/1.0/KneePitch_0.10.stl scale=0.1 0.1 0.1; visual mesh filename=package://pepper_meshes/meshes/1.0/KneePitch_0.10.stl scale=0.1 0.1 0.1
- link WheelB_link: geometry collision mesh filename=package://pepper_meshes/meshes/1.0/WheelB_0.10.stl scale=0.1 0.1 0.1; visual mesh filename=package://pepper_meshes/meshes/1.0/WheelB_0.10.stl scale=0.1 0.1 0.1
- link WheelFL_link: geometry collision mesh filename=package://pepper_meshes/meshes/1.0/WheelFL_0.10.stl scale=0.1 0.1 0.1; visual mesh filename=package://pepper_meshes/meshes/1.0/WheelFL_0.10.stl scale=0.1 0.1 0.1
- link WheelFR_link: geometry collision mesh filename=package://pepper_meshes/meshes/1.0/WheelFR_0.10.stl scale=0.1 0.1 0.1; visual mesh filename=package://pepper_meshes/meshes/1.0/WheelFR_0.10.stl scale=0.1 0.1 0.1
- link l_wrist: geometry collision mesh filename=package://pepper_meshes/meshes/1.0/LWristYaw_0.10.stl scale=0.1 0.1 0.1; visual mesh filename=package://pepper_meshes/meshes/1.0/LWristYaw_0.10.stl scale=0.1 0.1 0.1
- link r_wrist: geometry collision mesh filename=package://pepper_meshes/meshes/1.0/RWristYaw_0.10.stl scale=0.1 0.1 0.1; visual mesh filename=package://pepper_meshes/meshes/1.0/RWristYaw_0.10.stl scale=0.1 0.1 0.1
- link torso: geometry collision mesh filename=package://pepper_meshes/meshes/1.0/Torso_0.10.stl scale=0.1 0.1 0.1; visual mesh filename=package://pepper_meshes/meshes/1.0/Torso_0.10.stl scale=0.1 0.1 0.1
